File: wer3.kicad_pcb (KiCad board)
At the start: 2 copper layers, 61.2 x 129 mm, 65 parts, among them IC1 PCF8574T, J1 Conn_01x02_Pin, J10 Conn_01x02_Pin, J11 Conn_01x02_Pin, J12 Conn_01x02_Pin, J13 Conn_01x02_Pin, J14 Conn_01x02_Pin, J15 Conn_01x02_Pin, J16 Conn_01x02_Pin, J17 Conn_01x02_Pin, J18 Conn_01x02_Pin, J19 Conn_01x04_Socket, J2 Conn_01x02_Pin, J4 Conn_01x02_Pin, J5 Conn_01x02_Pin, J6 Conn_01x02_Pin, J7 Conn_01x02_Pin, J8 Conn_01x02_Pin, J9 Conn_01x02_Pin, U1 S102S02, U1b1 S102S02, U2 S102S02, U2b1 S102S02, U3 S102S02, U3b1 S102S02, U4 S102S02, U4b1 S102S02, U5 S102S02, U5b1 S102S02, U6 S102S02, U6b1 S102S02, U7 S102S02, U7b1 S102S02, U8 S102S02, U8b1 S102S02

Commit message: update
Parts:
- added R12: 10k, Resistor_SMD:R_0603_1608Metric, F.Cu at (120.2, 96.0)
- added R13: 10k, Resistor_SMD:R_0603_1608Metric, F.Cu at (118.6, 96.0)
- moved C1 3.36 mm to (115.4, 96.0), turned to 90 degrees
- moved C2 2.98 mm to (113.8, 96.0), turned to 90 degrees
- moved R14 2.24 mm to (117.0, 96.0), turned to 90 degrees
- moved C3 1.58 mm to (112.2, 96.0), turned to 90 degrees
- moved J19 1.08 mm to (119.8, 104.1)
- moved JP2 0.20 mm to (115.0, 74.4), turned to 180 degrees
- moved JP3 0.20 mm to (115.0, 77.1), turned to 180 degrees
- turned JP1 to 180 degrees
- renumbered C3 to C2, C2 to C3, J11 to J10, J12 to J11, J13 to J12, J14 to J13, J15 to J14, J16 to J15, J17 to J16, J18 to J17, J4 to J3, J5 to J4, J6 to J5, J7 to J6, J8 to J7, J9 to J8, J10 to J9, R9 to R11, R12 to R14, R11 to R9
Connections:
- IC1 pad 1: Net-(IC1-A0) -> A0
- IC1 pad 2: Net-(IC1-A1) -> A1
- IC1 pad 3: Net-(IC1-A2) -> A2
- JP1 pad 1: 5V -> A0
- JP1 pad 2: Net-(IC1-A0) -> 5V
- JP2 pad 1: 5V -> A1
- JP2 pad 2: Net-(IC1-A1) -> 5V
- JP3 pad 1: 5V -> A2
- JP3 pad 2: Net-(IC1-A2) -> 5V
- R10 pad 1: Net-(IC1-A1) -> A1
- R11 pad 1: Net-(IC1-A2) -> A2
- R9 pad 1: Net-(IC1-A0) -> A0
Routing:
- net Gnd: track 68.2 -> 46.3 mm
- net Net-(IC1-A0): track 16.4 -> 0.00 mm, vias 2 -> 0
- net A0: track 0.00 -> 16.0 mm, vias 0 -> 2
- net Net-(IC1-A1): track 13.6 -> 0.00 mm, vias 2 -> 0
- net A1: track 0.00 -> 12.9 mm, vias 0 -> 2
- net Net-(IC1-A2): track 10.5 -> 0.00 mm, vias 2 -> 0
- net A2: track 0.00 -> 9.79 mm, vias 0 -> 2
- net out1: track 49.2 -> 47.8 mm
- net out2: track 40.7 -> 39.3 mm
- net SDA: track 20.3 -> 21.6 mm
- net SCL: track 26.1 -> 27.1 mm
- net out5: track 52.2 -> 51.7 mm
- added copper zone on F.Cu, net Gnd
Other:
- outline, holes or cut-outs redrawn
