File: wer3.kicad_sch (KiCad schematic)
At the start: 65 parts, among them IC1 PCF8574T, J1 Conn_01x02_Pin, J10 Conn_01x02_Pin, J11 Conn_01x02_Pin, J12 Conn_01x02_Pin, J13 Conn_01x02_Pin, J14 Conn_01x02_Pin, J15 Conn_01x02_Pin, J16 Conn_01x02_Pin, J17 Conn_01x02_Pin, J18 Conn_01x02_Pin, J19 Conn_01x04_Socket, J2 Conn_01x02_Pin, J4 Conn_01x02_Pin, J5 Conn_01x02_Pin, J6 Conn_01x02_Pin, J7 Conn_01x02_Pin, J8 Conn_01x02_Pin, J9 Conn_01x02_Pin, U1 S102S02, U1b1 S102S02, U2 S102S02, U2b1 S102S02, U3 S102S02, U3b1 S102S02, U4 S102S02, U4b1 S102S02, U5 S102S02, U5b1 S102S02, U6 S102S02, U6b1 S102S02, U7 S102S02, U7b1 S102S02, U8 S102S02, U8b1 S102S02

Commit message: update
Parts:
- added R12, R13: 10k, Resistor_SMD:R_0603_1608Metric, symbol Device:R
- renumbered C3 to C2, C2 to C3, J11 to J10, J12 to J11, J13 to J12, J14 to J13, J15 to J14, J16 to J15, J17 to J16, J18 to J17, J4 to J3, J5 to J4, J6 to J5, J7 to J6, J8 to J7, J9 to J8, J10 to J9, R9 to R11, R12 to R14, R11 to R9
Connections:
- net 5V: now also JP1.2 (B), JP2.2 (B), JP3.2 (B), R12.1, R13.1; no longer JP1.1 (A), JP2.1 (A), JP3.1 (A)
- net SCL: now also R13.2
- net SDA: now also R12.2
- net A2: now reaches IC1.3 (A2), R11.1
- net A2: now also JP3.1 (A); no longer JP3.2 (B)
- net A1: now reaches IC1.2 (A1), R10.1
- net A1: now also JP2.1 (A); no longer JP2.2 (B)
- net A0: now reaches IC1.1 (A0), R9.1
- net A0: now also JP1.1 (A); no longer JP1.2 (B)
Other:
- moved on the sheet: C1, C2, C3, IC1, JP1, JP2, JP3, R10, R11, R14, R9
